File: PropositionRoutage/Routage.kicad_pcb (KiCad board)
At the start: 2 copper layers, 110 x 100 mm, 52 parts, among them J2 Conn_01x02, J3 Conn_01x03, Q1 2N2907, Q10 TIP32, Q11 BD138, Q12 TIP31, Q13 2N2222, Q2 2N2907, Q3 2N2907, Q4 2N2222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

Commit message: Proposition Routage
Parts:
- moved R14 29.9 mm to (94.5, 84.6)
- moved R15 29.9 mm to (84.3, 89.7)
- moved Q6 16.6 mm to (95.0, 75.2)
- moved Q7 14.2 mm to (69.6, 84.3)
- moved C3 12.3 mm to (82.3, 71.6), turned to 270 degrees
- moved D2 9.67 mm to (74.9, 55.9), turned to 180 degrees
- moved R8 9.49 mm to (106.7, 67.1)
- moved Q12 9.24 mm to (107.7, 46.7), turned to 180 degrees
- moved C9 9.16 mm to (104.1, 31.8), turned to 90 degrees
- moved Q4 9.16 mm to (103.1, 91.9), turned to 225 degrees
- moved C7 5.36 mm to (117.9, 75.7), turned to 0 degrees
- moved C6 5.25 mm to (117.9, 66.0), turned to 0 degrees
- moved R2 5.24 mm to (72.4, 91.4)
- moved Q5 5.08 mm to (101.6, 104.1), turned to 150 degrees
- moved C10 4.57 mm to (114.8, 35.6), turned to 0 degrees
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Routing:
- net -12V: track 7.65 -> 308.0 mm, vias 0 -> 2
- net +12V: track 74.2 -> 206.7 mm
- net Net-(C2-Pad1): track 0.00 -> 98.4 mm
- net /U1-pp: track 0.00 -> 90.5 mm, vias 0 -> 1
- net /ib2: track 0.00 -> 68.4 mm
- net /ic1: track 0.00 -> 62.5 mm
- net Net-(Q6-Pad1): track 0.00 -> 55.8 mm
- net Net-(Q6-Pad2): track 0.00 -> 37.4 mm
- net /ib1: track 0.00 -> 36.7 mm, vias 0 -> 1
- net /iR11: track 0.00 -> 30.4 mm
- net /iC3: track 0.00 -> 28.3 mm, vias 0 -> 1
- net /iR12: track 0.00 -> 23.1 mm
- net Net-(Q8-Pad2): track 0.00 -> 22.9 mm
- net Net-(Q6-Pad3): track 0.00 -> 22.8 mm
- net /ie1: track 0.00 -> 19.8 mm
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- added copper zone on B.Cu, net /iR17
- added copper zone on B.Cu, net GND
Other:
- board text added: "PIQUERAS DUMAS 15/04/2020 PCB Bottom"
- board text added: "PIQUERAS DUMAS 15/04/2020 PCB Top"
