File: PropositionRoutage/Routage.kicad_pcb (KiCad board)
At the start: 2 copper layers, 110 x 100 mm, 52 parts, among them J2 Conn_01x02, J3 Conn_01x03, Q1 2N2907, Q10 TIP32, Q11 BD138, Q12 TIP31, Q13 2N2222, Q2 2N2907, Q3 2N2907, Q4 2N2222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

Commit message: --all
Parts:
- moved Q8 10.1 mm to (77.5, 59.1)
- moved C1 7.73 mm to (59.7, 99.1)
- moved R16 6.98 mm to (63.5, 55.2)
- moved D2 6.87 mm to (69.2, 59.7), turned to 270 degrees
- moved R9 3.70 mm to (59.1, 74.3)
- moved R3 3.42 mm to (29.2, 95.9)
- moved D1 3.24 mm to (71.8, 43.8)
- moved Q2 3.24 mm to (34.9, 94.6), turned to 270 degrees
- moved Q7 3.06 mm to (69.8, 81.3)
- moved R4 1.91 mm to (49.5, 74.3)
- moved R7 1.91 mm to (66.0, 76.8)
- moved R17 1.27 mm to (85.1, 54.6)
- moved R12 1.27 mm to (83.8, 39.4)
- moved C10 0.13 mm to (114.9, 35.6)
Routing:
- net /ie1: track 19.8 -> 49.0 mm
- net /iR17: track 0.00 -> 19.9 mm
- net +12V: track 206.7 -> 216.6 mm
- net Net-(C2-Pad1): track 98.4 -> 88.6 mm
- net Net-(Q8-Pad2): track 22.9 -> 13.7 mm
- net /ib1: track 36.7 -> 29.5 mm, vias 1 -> 0
- net /iC3: track 28.3 -> 22.4 mm, vias 1 -> 0
- net /ib2: track 68.4 -> 62.8 mm
- net Net-(Q7-Pad3): track 14.3 -> 11.1 mm
- net Net-(Q6-Pad2): track 37.4 -> 34.3 mm
- net /U1-Q13: track 13.5 -> 11.4 mm
- net /jackcp: track 14.1 -> 16.0 mm
- net Net-(Q6-Pad3): track 22.8 -> 21.1 mm
- net /iR12: track 23.1 -> 21.8 mm
- net /U1-pp: track 90.5 -> 91.6 mm
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- added copper zone on B.Cu, net +12V
- added copper zone on B.Cu, net -12V
- removed copper zone on B.Cu, net /iR17
