File: Routage/Routage.sch (KiCad schematic (older format))
At the start: 52 parts, among them J2 Conn_01x02, J3 Conn_01x03, Q1 2N2907, Q10 TIP32, Q11 BD138, Q12 TIP31, Q13 2N2222, Q2 2N2907, Q3 2N2907, Q4 2N2222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

Commit message: Proposition Routage
Parts:
- removed HS3: Heatsink, CmpAmpliAudio:Heatsink_Fischer_SK104-STC-STIC_35x13mm_2xDrill2.5mm, symbol Mechanical:Heatsink
- added R14: R, CmpAmpliAudio:R_Axial_DIN0207_L6.3mm_D2.5mm_P10.16mm_Horizontal, symbol Device:R
- C11, C5, C7: footprint (none) -> CmpAmpliAudio:C_Rect_L7.2mm_W3.5mm_P5.00mm_FKS2_FKP2_MKS2_MKP2
- C9: renamed from C8; footprint (none) -> CmpAmpliAudio:C_Rect_L7.2mm_W3.5mm_P5.00mm_FKS2_FKP2_MKS2_MKP2
- R1, R10, R13, R15, R16, R17, R2, R3, R4, R5, R6, R7, R8, R9: footprint (none) -> CmpAmpliAudio:R_Axial_DIN0207_L6.3mm_D2.5mm_P10.16mm_Horizontal
- R11, R12: footprint (none) -> CmpAmpliAudio:R_Axial_DIN0516_L15.5mm_D5.0mm_P20.32mm_Horizontal
- U1: footprint (none) -> CmpAmpliAudio:Relais_112LMH2
- renumbered C9 to C8
Connections:
- net GND: now also J2.1 (Pin_1); no longer J2.2 (Pin_2)
- net U1-J2: now also J2.2 (Pin_2); no longer J2.1 (Pin_1)
- net U1-pp: now also R14.1; no longer Q2.1 (C), Q2.2 (B), R15.1, R3.1
- new net ib2: Q2.1 (C), Q2.2 (B), R14.2, R15.1, R3.1
